Commit message: joes final nav2 push

File: src/g1_description/urdf/g1_29dof_mode_15_brainco_hand.urdf (robot description, URDF)
Before this commit: robot g1_29dof_gazebo, 36 links, 35 joints
Joints:
- joint mid360_joint: origin xyz=0.0002835 0.00003 0.41618 rpy=0 0.04014257279586953 0 -> xyz=0.0002835 0.00003 0.41618 rpy=0 0.4014257279586953 0
